File: 0004_Heart_Rate_Module_MAX30102.kicad_sch (KiCad schematic)
At the start: 7 parts, among them U2 MAX30102EFD+, U3 MAX8511EXK18

Commit message: Add files via upload
Parts:
- removed U3: MAX8511EXK18, 21-0076E, symbol MAX8511EXK18:MAX8511EXK18
- added C2: 4,7uF, Capacitor_SMD:C_0603_1608Metric, symbol Device:C_Small
- added C2 (x7): 0,10uF, Capacitor_SMD:C_0603_1608Metric, symbol Device:C_Small
- added D1: LED, LED_SMD:LED_0603_1608Metric, symbol Device:LED
- added IC1: MAX8511EXK18+T, memin:SOT65P210X110-5N, symbol MAX8511EXK18+T:MAX8511EXK18+T
- added R1, R2: 1k, Resistor_SMD:R_0603_1608Metric, symbol Device:R
- added R1: 470r, Resistor_SMD:R_0603_1608Metric, symbol Device:R
- added U3: ~, Moduler_:pin_header, symbol moduler_pin:air
- added U4: PCA9306, Package_SO:VSSOP-8_2.3x2mm_P0.5mm, symbol Interface:PCA9306
- added U5: SN74LVC1T45DBV, Package_TO_SOT_SMD:SOT-23-6, symbol Logic_LevelTranslator:SN74LVC1T45DBV
- C1, C2: footprint (none) -> Capacitor_SMD:C_0603_1608Metric
- R1, R2, R3: footprint (none) -> Resistor_SMD:R_0603_1608Metric
Connections:
- net +1V8: now also C2.1, C2.1, C2.1, C2.1, IC1.5 (OUT), R1.1, R2.1, U4.2 (VREF1), U5.1 (VCCA)
- net GND: now also C2.2, C2.2, C2.2, C2.2, C2.2, C2.2, C2.2, C2.2, D1.1 (K), IC1.2 (GND), U3.9, U4.1 (GND), U5.2 (GND)
- net INT: now also U3.12, U5.4 (B); no longer U2.13 (~{INT})
- net SCL: now also R2.2, U3.5, U4.6 (SCL2); no longer R1.2, U2.2 (SCL)
- net SDA: now also R1.2, U3.6, U4.5 (SDA2); no longer R2.2, U2.3 (SDA)
- net +5V renamed +3V3
- net +3V3: now also C2.1, C2.1, C2.1, C2.1, IC1.1 (IN), IC1.3 (~{SHDN}), R1.1, U3.8, U4.7 (VREF2), U4.8 (EN), U5.5 (DIR), U5.6 (VCCB)
- new net: D1.2 (A), R1.2
- new net INT_: U2.13 (~{INT}), U5.3 (A)
- new net SCL_: R1.2, U2.2 (SCL), U4.3 (SCL1)
- new net SDA_: R2.2, U2.3 (SDA), U4.4 (SDA1)
- no-connect marks 7 -> 19
Other:
- note added: "AIR PIN"
- note added: "BUCK"
- note added: "I2C PULLUPS"
- note added: "SENSOR"
- note added: "TRANSLATOR"
- moved on the sheet: C1, C2, R1, R2, R3, U2
